File: MacroPad/MacroPad/MacroPad.kicad_sch (KiCad schematic)
At the start: 24 parts

Commit message: Add footprints for all components on macropad
Parts:
- C1, C2: value (none) -> 22pF; footprint (none) -> Capacitor_SMD:C_0805_2012Metric
- C3: value (none) -> 1uF; footprint (none) -> Capacitor_SMD:C_0805_2012Metric
- C4: value (none) -> 0.1uF; footprint (none) -> Capacitor_SMD:C_0805_2012Metric
- C5, C6: footprint (none) -> Capacitor_SMD:C_0805_2012Metric
- C7: value (none) -> 10uF; footprint (none) -> Capacitor_SMD:C_0805_2012Metric
- D1: value (none) -> D_Small; footprint (none) -> Diode_SMD:D_SOD-123
- D2, D3, D4: footprint (none) -> Diode_SMD:D_SOD-123
- F1: value (none) -> 500mA; footprint (none) -> Fuse:Fuse_1206_3216Metric
- MX1: value (none) -> MX-NoLED; footprint (none) -> MX_Alps_Hybrid:MX-1U-NoLED
- MX2, MX3, MX4: footprint (none) -> MX_Alps_Hybrid:MX-1U-NoLED
- R1, R2: value (none) -> 10k; footprint (none) -> Resistor_SMD:R_0805_2012Metric
- R3, R4: value (none) -> 22; footprint (none) -> Resistor_SMD:R_0805_2012Metric
- SW1: value (none) -> SW_Push
- U1: value (none) -> ATmega32U4-AU; footprint (none) -> Package_QFP:TQFP-44_10x10mm_P0.8mm
- USB1: value (none) -> Molex-0548190589
- Y1: value (none) -> 16MHz

Commit message: Add QMK layout files for firmware
Parts:
- SW1: footprint (none) -> random-keyboard-parts:SKQG-1155865
- USB1: footprint (none) -> random-keyboard-parts:Molex-0548190589
- Y1: footprint (none) -> Crystal:Crystal_SMD_3225-4Pin_3.2x2.5mm
